File: Hardware/PiGarage.kicad_sch (KiCad schematic)
At the start: 73 parts, among them J1 Conn_02x03_Odd_Even, J2 Conn_02x02_Counter_Clockwise, J3 PJ-320B, J4 Conn_02x20_Odd_Even, Q1 MMBT3904, U1 PCM5122PWR, U2 TPS54560BQDDARQ1, U3 TL431DBZ, U4 AP2112K-3.3, U5 Optocoupler_DC_PhotoNPN_AKEC, U6 Optocoupler_DC_PhotoNPN_AKEC, U7 Optocoupler_DC_PhotoNPN_AKEC, U8 Optocoupler_DC_PhotoNPN_AKEC, U9 ADS1115IDGS

Commit message: v0.2
- Buck converter redesigned with TI WEBENCH (7-16V in, 5V/5A, 1.1MHz fsw)
- New inductor: FXL0630-2R2-M (2.2µH, 10A Isat, 15mΩ DCR)
- New catch diode: B560C-13-F (SMC package for better thermals)
- Added AO4407A P-FET reverse polarity protection
- Replaced 4× LTV-817S with 1× LTV-847S quad optocoupler
- Switched ADS1115 back to VSSOP (IDGSR) from QFN
- All passives upgraded from 0402 to 0603 for hand-solder friendliness
- Fixed DAC pin connections (BCM21 for DIN, XSMT to 3.3VA)
- Fixed ADC pull-up topology for correct voltage divider operation
- Merged AGND into GND (shared ground per PCM5122 datasheet)
- Added GND via stitching (65 vias)
- Updated all 3D model paths for KiCad 10
- Updated BOM, design notes, and README
Parts:
- removed C3: 1µF, Capacitor_SMD:C_0402_1005Metric, symbol Device:C
- removed NT1: NetTie_2, NetTie:NetTie-2_SMD_Pad0.5mm, symbol Device:NetTie_2
- removed R14, R17, R18, R26: 10kΩ, Resistor_SMD:R_0402_1005Metric, symbol Device:R
- removed R27, R28: 4.7kΩ, Resistor_SMD:R_0402_1005Metric, symbol Device:R
- removed U5, U6, U7, U8: Optocoupler_DC_PhotoNPN_AKEC, FOD817BSD:SOIC254P1016X385-4N, symbol Isolator:Optocoupler_DC_PhotoNPN_AKEC
- removed U9: ADS1115IDGS, ADS1115IRUGR:IC_ADS1115IRUGR, symbol PCM_JLCPCB-Extended:ADC, ADS1115IDGS
- added C12, C16, C22: 10µF, Capacitor_SMD:C_0603_1608Metric, symbol Device:C
- added C21: 0.1µF, Capacitor_SMD:C_0603_1608Metric, symbol Device:C
- added C30, C31, C32, C33: 100nF, Capacitor_SMD:C_0603_1608Metric, symbol Device:C
- added C6: 47µF, Capacitor_SMD:C_1206_3216Metric, symbol Device:C
- added Q1: AO4407A, SOIC127P600X175:SOIC127P600X175-8N, symbol AO4407A:AO4407A
- added R19, R20, R21, R22: 4.7kΩ, Resistor_SMD:R_0603_1608Metric, symbol Device:R
- added U5: ADS1115IDGSR, ADS1115IDGSR:SOP50P490X110-10N, symbol ADS1115IDGSR:ADS1115IDGSR
- added U6: LTV-847S, Package_DIP:SMDIP-16_W9.53mm, symbol Isolator:LTV-847S
- C1: value 10µF -> 4.7µF; footprint Capacitor_SMD:C_0805_2012Metric -> Capacitor_SMD:C_1206_3216Metric
- C10: renamed from C9; footprint Capacitor_SMD:C_0402_1005Metric -> Capacitor_SMD:C_0603_1608Metric
- C11: renamed from C10; footprint Capacitor_SMD:C_0805_2012Metric -> Capacitor_SMD:C_0603_1608Metric
- C13: renamed from C20; value 100nF -> 0.1µF; footprint Capacitor_SMD:C_0402_1005Metric -> Capacitor_SMD:C_0603_1608Metric
- C14: renamed from C16; value 10µF -> 2.2µF; footprint Capacitor_SMD:C_0805_2012Metric -> Capacitor_SMD:C_0603_1608Metric
- C15: renamed from C17; value 1µF -> 2.2µF; footprint Capacitor_SMD:C_0402_1005Metric -> Capacitor_SMD:C_0603_1608Metric
- C17: renamed from C11; value 100nF -> 0.1µF; footprint Capacitor_SMD:C_0402_1005Metric -> Capacitor_SMD:C_0603_1608Metric
- C18: renamed from C12; footprint Capacitor_SMD:C_0805_2012Metric -> Capacitor_SMD:C_0603_1608Metric
- C19: renamed from C13; value 100nF -> 0.1µF; footprint Capacitor_SMD:C_0402_1005Metric -> Capacitor_SMD:C_0603_1608Metric
- C2: footprint Capacitor_SMD:C_0402_1005Metric -> Capacitor_SMD:C_0603_1608Metric
- C20: renamed from C14; footprint Capacitor_SMD:C_0805_2012Metric -> Capacitor_SMD:C_0603_1608Metric
- C25: renamed from C21; footprint Capacitor_SMD:C_0402_1005Metric -> Capacitor_SMD:C_0603_1608Metric
- C26: renamed from C15; footprint Capacitor_SMD:C_0402_1005Metric -> Capacitor_SMD:C_0603_1608Metric
- C27: renamed from C22; footprint Capacitor_SMD:C_0402_1005Metric -> Capacitor_SMD:C_0603_1608Metric
- C28: renamed from C25; footprint Capacitor_SMD:C_0402_1005Metric -> Capacitor_SMD:C_0603_1608Metric
- C29: renamed from C23; footprint Capacitor_SMD:C_0402_1005Metric -> Capacitor_SMD:C_0603_1608Metric
- C3: renamed from C5; value 47pF -> 1.8nF; footprint Capacitor_SMD:C_0402_1005Metric -> Capacitor_SMD:C_0603_1608Metric
- C4: renamed from C6; value 1nF -> 8.2pF; footprint Capacitor_SMD:C_0402_1005Metric -> Capacitor_SMD:C_0603_1608Metric
- C5: renamed from C4; footprint Capacitor_SMD:CP_Elec_6.3x5.7 -> Capacitor_SMD:C_1206_3216Metric
- C7: renamed from C8; footprint Capacitor_SMD:C_0805_2012Metric -> Capacitor_SMD:C_1206_3216Metric
- C8: renamed from C7; footprint Capacitor_SMD:C_0805_2012Metric -> Capacitor_SMD:C_0603_1608Metric
- C9: renamed from C24; footprint Capacitor_SMD:C_0402_1005Metric -> Capacitor_SMD:C_0603_1608Metric
- D1: value D_TVS -> SMBJ18CA; footprint Diode_SMD:D_SMB -> Diode_SMD:D_SMC
- D2: renamed from D3; value D_Schottky -> B560C-13-F; footprint Diode_SMD:D_SMA -> B560C:SMC_L7.1-W6.2-LS8.1-RD
- D3: renamed from D2; value D_Schottky_Dual_CommonCathode_AKA -> BAT54CLT1G
- L1: value 10µH -> 2.2µH; footprint Inductor_SMD:L_Sunlord_MWSA1204S-100 -> FXL0630:IND-SMD_L7.0-W6.6
- Q2: renamed from Q1; footprint Package_TO_SOT_SMD:SOT-23 -> Package_TO_SOT_SMD:TSOT-23
- R1: renamed from R4; value 15kΩ -> 23.7kΩ; footprint Resistor_SMD:R_0402_1005Metric -> Resistor_SMD:R_0603_1608Metric
- R10: renamed from R8; footprint Resistor_SMD:R_0402_1005Metric -> Resistor_SMD:R_0603_1608Metric
- R11: renamed from R21; footprint Resistor_SMD:R_0402_1005Metric -> Resistor_SMD:R_0603_1608Metric
- R12: renamed from R6; footprint Resistor_SMD:R_0402_1005Metric -> Resistor_SMD:R_0603_1608Metric
- R13: renamed from R15; footprint Resistor_SMD:R_0402_1005Metric -> Resistor_SMD:R_0603_1608Metric
- R14: renamed from R16; footprint Resistor_SMD:R_0402_1005Metric -> Resistor_SMD:R_0603_1608Metric
- R15: renamed from R22; footprint Resistor_SMD:R_0402_1005Metric -> Resistor_SMD:R_0603_1608Metric
- R16: renamed from R20; footprint Resistor_SMD:R_0402_1005Metric -> Resistor_SMD:R_0603_1608Metric
- R17: renamed from R24; footprint Resistor_SMD:R_0402_1005Metric -> Resistor_SMD:R_0603_1608Metric
- R18: renamed from R19; footprint Resistor_SMD:R_0402_1005Metric -> Resistor_SMD:R_0603_1608Metric
- R2: renamed from R1; value 200kΩ -> 80.6kΩ; footprint Resistor_SMD:R_0402_1005Metric -> Resistor_SMD:R_0603_1608Metric
- R23: renamed from R5; footprint Resistor_SMD:R_0402_1005Metric -> Resistor_SMD:R_0603_1608Metric
- R24: renamed from R7; footprint Resistor_SMD:R_0402_1005Metric -> Resistor_SMD:R_0603_1608Metric
- R25: renamed from R23; footprint Resistor_SMD:R_0402_1005Metric -> Resistor_SMD:R_0603_1608Metric
- R26: renamed from R25; footprint Resistor_SMD:R_0402_1005Metric -> Resistor_SMD:R_0603_1608Metric
- R3: renamed from R2; value 52.3kΩ -> 60.4kΩ; footprint Resistor_SMD:R_0402_1005Metric -> Resistor_SMD:R_0603_1608Metric
- R4: renamed from R3; value 10kΩ -> 11.5kΩ; footprint Resistor_SMD:R_0402_1005Metric -> Resistor_SMD:R_0603_1608Metric
- R5: renamed from R9; footprint Resistor_SMD:R_0402_1005Metric -> Resistor_SMD:R_0603_1608Metric
- R6: renamed from R10; footprint Resistor_SMD:R_0402_1005Metric -> Resistor_SMD:R_0603_1608Metric
- R7: renamed from R11; footprint Resistor_SMD:R_0402_1005Metric -> Resistor_SMD:R_0603_1608Metric
- R8: renamed from R12; footprint Resistor_SMD:R_0402_1005Metric -> Resistor_SMD:R_0603_1608Metric
- R9: renamed from R13; footprint Resistor_SMD:R_0402_1005Metric -> Resistor_SMD:R_0603_1608Metric
- U3: renamed from U1; footprint PCM5122PWR:SOP65P640X120-28N -> Package_SO:TSSOP-28_4.4x9.7mm_P0.65mm
- renumbered C18 to C23, C19 to C24, U2 to U1, U3 to U2
Connections:
- net +3.3V: now also C18.2, U3.24 (ADR1), U3.25 (XSMT), C33.1, R19.2, R20.2, R21.2, R22.2; no longer C29.1
- net +3.3VA: now also C11.2, C20.2, C21.1, C22.2
- net +5V: now also C6.1
- net +VBAT: now also Q1.1, Q1.2, Q1.3; no longer C1.1, D1.1 (A1), U1.2 (VIN)
- net AIN0: now also R23.2, R19.1; no longer R23.1
- net AIN1: now also R24.2, R20.1; no longer R24.1
- net AIN2: now also R25.2, R21.1; no longer R25.1
- net AIN3: now also R26.2, R22.1; no longer R26.1
- net BCM17: now also U6.12
- net BCM2: now also U5.9 (SDA)
- net BCM22: now also U6.14
- net BCM24: now also U6.10
- net BCM27: now also U6.16
- net BCM3: now also U5.10 (SCL)
- net GND: now also C10.1, C11.1, C13.1, C14.2, C17.2, C18.1, C19.2, C20.1, C23.1, C24.2, C29.1, C9.2, J3.3, U3.16 (ADR2), U3.17 (MODE1), U3.20 (SCK), U3.27 (DGND), U3.9 (AGND), U4.2 (GND), C12.1, C16.1, C21.2, C22.1, C30.2, C31.2, C32.2, C6.2, Q1.4, U5.1 (ADDR), U5.3 (GND), U6.11, U6.13, U6.15, U6.2, U6.4, U6.6, U6.8, U6.9; no longer C29.2
- net at C13.2, U3.26 (LDOO): now also C12.2
- net at C25.1, R15.2: now also U6.1
- net at C28.1, R18.2: now also U6.7
- net at C26.1, R16.2: now also U6.3
- net at C27.1, R17.2: now also U6.5
- net at C3.1, R1.1: no longer U1.6 (COMP)
- net at C4.1, R1.2: now also U1.6 (COMP)
- net BCM21: now reaches J4.40 (Pin_40)
- net BCM21: now also U3.22 (DIN)
- removed net AGND: C11.1, C13.1, C14.2, C18.2, C20.2, C23.1, C24.2, C9.2, J3.3, U3.10 (VCOM), U3.17 (MODE1), U3.20 (SCK), U3.27 (DGND), U3.3 (CPGND), U3.9 (AGND), U4.2 (GND)
- net BCM20: no longer names the net of J4.38 (Pin_38)
- net BCM20: no longer U3.22 (DIN)
- new net: C32.1, R26.1, U5.7 (AIN3)
- new net: C1.1, D1.1 (A1), Q1.5, Q1.6, Q1.7, Q1.8, U1.2 (VIN)
- new net: C31.1, R25.1, U5.6 (AIN2)
- new net: C29.2, R23.1, U5.4 (AIN0)
- new net: C30.1, R24.1, U5.5 (AIN1)
- new net: C33.2, U5.8 (VDD)
- new net: C16.2, U3.10 (VCOM)
Other:
- moved on the sheet: C1, C10, C11, C13, C17, C18, C2, C20, C23, C24, C25, C26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

Commit message: Add thermal pad to D2 and remap GPIO sense pins
- Added exposed copper thermal pad (GND, pad 3) with 4 thermal vias to
  D2 (B560C catch diode) footprint for improved heat dissipation at 5A
- Remapped optoisolator GPIO assignments for cleaner PCB trace routing:
    BCM17 = ACC, BCM22 = REV, BCM27 = ILL, BCM24 = AUX
- Updated power_latch.py PIN_ACC 27 → 17 to match new assignment
- Updated design-notes and GPIO allocation table
- Cleaned up stale SVG exports from Images/
Connections:
- net BCM17: now also U6.16; no longer U6.12
- net BCM22: now also U6.12; no longer U6.14
- net BCM27: now also U6.14; no longer U6.16
Changed lines of the file:
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@@
 		)
 	)
-	(label "BCM27"
+	(label "BCM17"
 		(at 68.58 187.96 0)
 		(effects
@@
 		)
 	)
-	(label "BCM17"
+	(label "BCM22"
 		(at 64.77 257.81 0)
 		(effects
@@
 		)
 	)
-	(label "BCM22"
+	(label "BCM27"
 		(at 66.04 222.25 0)
 		(effects

Commit message: Fix D1 footprint: D_SMC (DO-214AB) → D_SMB (DO-214AA)
SMBJ18CA ships in SMB (DO-214AA) package; the SMC footprint had
~60% larger pads and courtyard, causing JLCPCB preview mismatch.
Updated pad positions (±3.4 → ±2.15 mm), pad size (3.3×2.5 →
2.5×2.3 mm), courtyard, silkscreen, fab outline, and 3D model to
match KiCad Diode_SMD:D_SMB. Re-routing of D1 connections required
in KiCad after this change.
Parts:
- D1: footprint Diode_SMD:D_SMC -> Diode_SMD:D_SMB
Changed lines of the file:
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@@
 			)
 		)
-		(property "Footprint" "Diode_SMD:D_SMC"
+		(property "Footprint" "Diode_SMD:D_SMB"
 			(at 124.46 27.94 0)
 			(hide yes)

Commit message: Update BOM and design notes: swap 0402 passives to 0603
All affected resistors and decoupling caps updated to 0603 footprint
equivalents to support hand soldering. LCSC part numbers, MPNs, and
specs updated throughout design-notes.txt. Schematic symbol properties
updated with new 0603 LCSC numbers. BOM tracking CSV added.
Parts:
- C13, C17, C19, C21: LCSC (none) -> C14663; MPN (none) -> CC0603KRX7R9BB104; Manufacturer (none) -> Yageo
- R10: LCSC (none) -> C25803; MPN (none) -> 0603WAF1003T5E; Manufacturer (none) -> UNI-ROYAL(Uniroyal Elec)
- R11, R19, R20, R21, R22: LCSC (none) -> C23162; MPN (none) -> 0603WAF4701T5E; Manufacturer (none) -> UNI-ROYAL(Uniroyal Elec)
- R12, R6: LCSC (none) -> C31850; MPN (none) -> 0603WAF2202T5E; Manufacturer (none) -> UNI-ROYAL(Uniroyal Elec)
- R13, R14: LCSC (none) -> C23179; MPN (none) -> 0603WAF4700T5E; Manufacturer (none) -> UNI-ROYAL(Uniroyal Elec)
- R15, R16, R17, R18, R23, R24, R25, R26, R9: LCSC (none) -> C25804; MPN (none) -> 0603WAF1002T5E; Manufacturer (none) -> UNI-ROYAL(Uniroyal Elec)
- R5: LCSC (none) -> C23118; MPN (none) -> 0603WAF8452T5E; Manufacturer (none) -> UNI-ROYAL(Uniroyal Elec)
- R7: LCSC (none) -> C21190; MPN (none) -> 0603WAF1001T5E; Manufacturer (none) -> UNI-ROYAL(Uniroyal Elec)
- R8: LCSC (none) -> C25819; MPN (none) -> 0603WAF4702T5E; Manufacturer (none) -> UNI-ROYAL(Uniroyal Elec)
